File: elec/layout/dual/dual.kicad_pcb (KiCad board)
At the start: 2 copper layers, 9 parts

Commit message: build with latest
Parts:
- R1, R2, R3, R4: value 51Ω ±1% 62.5mW -> 47Ω ±1% 62.5mW
Connections:
- net scl renamed SCL
- R2 pad 1: p-1 -> p
- R4 pad 1: p -> p-1
